File: DCI_TP/DCI_TP.kicad_pcb (KiCad board)
At the start: 2 copper layers, 50 parts, among them Q1 12.288Mhz, U1 V_REG_LDOSMD, U2 V_REG_LDOSMD, U3 V_REG_LDOSMD

Commit message: New commit DCI
Se suben avances de PCB
Parts:
- removed JP1: M10, SparkFun-Connectors:1X10_LOCK
- removed U3: V_REG_LDOSMD, SparkFun-Sensors:SOT23-5
- removed VS1053: VS1033_1053SMD, SparkFun-DigitalIC:LQFP-48
- added JP2: M10, SparkFun_MP3_Breakout-VS1063:1X10, F.Cu at (135.8, 88.5)
- added U$12: 1.8V, SparkFun_MP3_Breakout-VS1063:SC70, F.Cu at (153.0, 97.4)
- added U$2: 2.8V, SparkFun_MP3_Breakout-VS1063:SC70, F.Cu at (130.7, 107.5)
- C1: value 100nF -> 10uF; footprint SparkFun-Capacitors:0402-CAP -> SparkFun_MP3_Breakout-VS1063:EIA3216
- C10: value 0.1uF -> 10nF; footprint SparkFun-Capacitors:0402-CAP -> SparkFun_MP3_Breakout-VS1063:0402-CAP
- C11: value 100nF -> 47nF; footprint SparkFun-Capacitors:0402-CAP -> SparkFun_MP3_Breakout-VS1063:0402-CAP
- C12: value 100nF -> 10nF; footprint SparkFun-Capacitors:0402-CAP -> SparkFun_MP3_Breakout-VS1063:0402-CAP
- C13, C14: value 18pF -> 100nF; footprint SparkFun-Capacitors:0402-CAP -> SparkFun_MP3_Breakout-VS1063:0402-CAP
- C15, C16, C17, C18, C23, C24, C9: footprint SparkFun-Capacitors:0402-CAP -> SparkFun_MP3_Breakout-VS1063:0402-CAP
- C19, C21: value 10nF -> 100nF; footprint SparkFun-Capacitors:0402-CAP -> SparkFun_MP3_Breakout-VS1063:0402-CAP
- C2, C7: value 100nF -> 0.1uF; footprint SparkFun-Capacitors:0402-CAP -> SparkFun_MP3_Breakout-VS1063:0402-CAP
- C20: value 47nF -> 100nF; footprint SparkFun-Capacitors:0402-CAP -> SparkFun_MP3_Breakout-VS1063:0402-CAP
- C22: value 0.1uF -> 100nF; footprint SparkFun-Capacitors:0402-CAP -> SparkFun_MP3_Breakout-VS1063:0402-CAP
- C3: value 100nF -> 18pF; footprint SparkFun-Capacitors:0402-CAP -> SparkFun_MP3_Breakout-VS1063:0402-CAP
- C4, C6: footprint SparkFun-Capacitors:EIA3216 -> SparkFun_MP3_Breakout-VS1063:EIA3216
- C5: value 10uF -> 0.1uF; footprint SparkFun-Capacitors:EIA3216 -> SparkFun_MP3_Breakout-VS1063:0402-CAP
- C8: value 0.1uF -> 18pF; footprint SparkFun-Capacitors:0402-CAP -> SparkFun_MP3_Breakout-VS1063:0402-CAP
- JP3: footprint SparkFun-Connectors:1X07 -> SparkFun_MP3_Breakout-VS1063:1X07
- JP4: footprint SparkFun-Capacitors:SJ_2S -> SparkFun_MP3_Breakout-VS1063:SJ_2S
- LED1: footprint SparkFun-LED:LED10MM -> SparkFun_MP3_Breakout-VS1063:LED-0603
- Q1: value 12.288Mhz -> 12.288MHz; footprint SparkFun-FreqCtrl:HC49U-V -> SparkFun_MP3_Breakout-VS1063:CRYSTAL-SMD-5X3
- R1: value 330 -> 1M; footprint SparkFun-Capacitors:0402-RES -> SparkFun_MP3_Breakout-VS1063:0402-RES
- R10, R16, R17, R2, R4, R5: footprint SparkFun-Capacitors:0402-RES -> SparkFun_MP3_Breakout-VS1063:0402-RES
- R11: value 20 -> 100k; footprint SparkFun-Capacitors:0402-RES -> SparkFun_MP3_Breakout-VS1063:0402-RES
- R12: value 10 -> 470; footprint SparkFun-Capacitors:0402-RES -> SparkFun_MP3_Breakout-VS1063:0402-RES
- R13: value 20 -> 470; footprint SparkFun-Capacitors:0402-RES -> SparkFun_MP3_Breakout-VS1063:0402-RES
- R14, R15: value 470 -> 100k; footprint SparkFun-Capacitors:0402-RES -> SparkFun_MP3_Breakout-VS1063:0402-RES
- R3: footprint SparkFun-Resistors:0402-RES -> SparkFun_MP3_Breakout-VS1063:0402-RES
- R6: value 1M -> 20; footprint SparkFun-Capacitors:0402-RES -> SparkFun_MP3_Breakout-VS1063:0402-RES
- R7: value 100k -> 10; footprint SparkFun-Capacitors:0402-RES -> SparkFun_MP3_Breakout-VS1063:0402-RES
- R8: value 100k -> 330; footprint SparkFun-Capacitors:0402-RES -> SparkFun_MP3_Breakout-VS1063:0402-RES
- R9: value 100k -> 20; footprint SparkFun-Capacitors:0402-RES -> SparkFun_MP3_Breakout-VS1063:0402-RES
- U1: value V_REG_LDOSMD -> 3.3V; footprint SparkFun-Sensors:SOT23-5 -> SparkFun_MP3_Breakout-VS1063:SOT23-5
- U2: value V_REG_LDOSMD -> VS1053; footprint SparkFun-Sensors:SOT23-5 -> SparkFun_MP3_Breakout-VS1063:LQFP-48
- moved R1 178.5 mm to (156.1, 103.7), turned to 90 degrees
- moved U2 167.4 mm to (146.0, 103.7)
- moved C8 165.6 mm to (161.2, 105.0), turned to 270 degrees
- moved U1 163.1 mm to (158.7, 112.6)
- moved LED1 161.5 mm to (132.0, 110.1), turned to 270 degrees
- moved C4 155.0 mm to (156.1, 97.4), turned to 270 degrees
- moved JP3 45.6 mm to (168.8, 111.4), turned to 90 degrees
- moved R14 34.5 mm to (166.3, 97.4), turned to 0 degrees
- moved R8 34.5 mm to (129.5, 110.1), turned to 180 degrees
- moved C2 30.7 mm to (130.7, 101.2), turned to 180 degrees
- moved R15 29.4 mm to (166.3, 99.9), turned to 0 degrees
- moved R3 29.2 mm to (142.0, 95.0), turned to 270 degrees
- moved C6 28.7 mm to (154.9, 112.6), turned to 90 degrees
- moved R7 27.8 mm to (134.5, 101.2), turned to 270 degrees
- moved JP4 26.0 mm to (135.8, 105.0)
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Connections:
- C10 pad 1: /CVDD -> Net-(C10-Pad1)
- C10 pad 2: GND -> /AGND
- C11 pad 1: /CVDD -> Net-(C11-Pad1)
- C11 pad 2: GND -> /AGND
- C12 pad 1: /CVDD -> Net-(C12-Pad1)
- C12 pad 2: GND -> /AGND
- C13 pad 1: Net-(C13-Pad1) -> /CVDD
- C14 pad 1: Net-(C14-Pad1) -> /CVDD
- C16 pad 1: /IOVDD -> /CVDD
- C17 pad 1: /IOVDD -> /AVDD
- C17 pad 2: GND -> /AGND
- C18 pad 1: /IOVDD -> /AVDD
- C18 pad 2: GND -> /AGND
- C19 pad 1: Net-(C19-Pad1) -> /AVDD
- C20 pad 1: Net-(C20-Pad1) -> /IOVDD
- C20 pad 2: /AGND -> GND
- C21 pad 1: Net-(C21-Pad1) -> /IOVDD
- C21 pad 2: /AGND -> GND
- C22 pad 1: Net-(C22-Pad1) -> /IOVDD
- C22 pad 2: /AGND -> GND
- C3 pad 1: /AVDD -> Net-(C3-Pad1)
- C3 pad 2: /AGND -> GND
- C4 pad A: /IOVDD -> /CVDD
- C6 pad A: /CVDD -> /IOVDD
- C8 pad 1: /IOVDD -> Net-(C8-Pad1)
- C9 pad 1: /AVDD -> Net-(C9-Pad1)
- Q1 pad 1: Net-(C13-Pad1) -> Net-(C8-Pad1)
- Q1 pad 2: Net-(C14-Pad1) -> (no net)
- R1 pad 1: /VCC -> Net-(C3-Pad1)
- R1 pad 2: Net-(LED1-PadA) -> Net-(C8-Pad1)
- R10 pad 1: /GPIO4 -> /GPIO3
- R11 pad 1: /RIGHT -> /GPIO2
- R11 pad 2: Net-(C19-Pad1) -> GND
- R12 pad 1: /GBUF -> Net-(R12-Pad1)
- R12 pad 2: Net-(C20-Pad1) -> /MICP
- R13 pad 1: /LEFT -> Net-(R13-Pad1)
- R13 pad 2: Net-(C21-Pad1) -> /LINEIN
- R14 pad 1: Net-(R14-Pad1) -> /GPIO4
- R14 pad 2: /MICP -> GND
- R15 pad 1: Net-(R15-Pad1) -> /GPIO5
- R15 pad 2: /LINEIN -> GND
- R16 pad 1: /GPIO1 -> /GPIO7
- R17 pad 1: /GPIO0 -> /GPIO6
- R2 pad 2: /RESET -> /RX
- R3 pad 1: /GPIO3 -> /GPIO1
- R4 pad 1: /GPIO2 -> /GPIO0
- R5 pad 2: /RX -> /RESET
- R6 pad 1: Net-(C13-Pad1) -> /RIGHT
- R6 pad 2: Net-(C14-Pad1) -> Net-(C10-Pad1)
- R7 pad 1: /GPIO6 -> /GBUF
- R7 pad 2: GND -> Net-(C11-Pad1)
- R8 pad 1: /GPIO7 -> /VCC
- R8 pad 2: GND -> Net-(LED1-PadA)
- R9 pad 1: /GPIO5 -> /LEFT
- R9 pad 2: GND -> Net-(C12-Pad1)
- U1 pad 2: /VCC -> GND
- U1 pad 3: GND -> /VCC
- U2 pad 1: /VCC -> Net-(R12-Pad1)
- U2 pad 2: /VCC -> /MICN
- U2 pad 3: /AGND -> /RESET
- U2 pad 4: Net-(U2-Pad4) -> /PWR_FLAG
- U2 pad 5: /AVDD -> /CVDD
Routing:
- net GND: track 0.00 -> 227.3 mm, vias 0 -> 1
- net /AGND: track 0.00 -> 109.9 mm
- net /VCC: track 0.00 -> 89.1 mm, vias 0 -> 1
- net /IOVDD: track 0.00 -> 63.4 mm, vias 0 -> 5
- net /CVDD: track 0.00 -> 63.3 mm, vias 0 -> 5
- net /LINEIN: track 0.00 -> 48.5 mm, vias 0 -> 1
- net /GPIO4: track 0.00 -> 42.0 mm, vias 0 -> 1
- net /RX: track 0.00 -> 38.2 mm, vias 0 -> 1
- net /AVDD: track 0.00 -> 34.8 mm, vias 0 -> 3
- net /CS: track 0.00 -> 32.5 mm, vias 0 -> 1
- net /GPIO7: track 0.00 -> 30.4 mm, vias 0 -> 1
- net /GPIO2: track 0.00 -> 29.7 mm, vias 0 -> 1
- net /TX: track 0.00 -> 28.6 mm, vias 0 -> 1
- net /GPIO6: track 0.00 -> 27.0 mm, vias 0 -> 1
- net /RIGHT: track 0.00 -> 26.0 mm, vias 0 -> 2
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