File: DCI_TP/DCI_TP.sch (KiCad schematic (older format))
At the start: 51 parts, among them Q1 12.288Mhz, U1 V_REG_LDOSMD, U2 V_REG_LDOSMD, U3 V_REG_LDOSMD

Commit message: New commit DCI
Se suben avances de PCB
Parts:
- removed JP1: M10\", SparkFun-Connectors:1X10_LOCK, symbol SparkFun-Connectors:M10LOCK
- removed LED1: Power, SparkFun-LED:LED10MM, symbol SparkFun-LED:LED10MM
- removed Q1: 12.288Mhz, SparkFun-FreqCtrl:HC49U-V, symbol DCI_TP-rescue:CRYSTALHC49U-V-adafruit
- removed U1, U2, U3: V_REG_LDOSMD, SparkFun-Sensors:SOT23-5, symbol SparkFun-PowerIC:V_REG_LDOSMD
- removed VS1053: VS1033_1053SMD, SparkFun-DigitalIC:LQFP-48, symbol SparkFun-DigitalIC:VS1033_1053SMD
- added JP1: M10\", SparkFun_MP3_Breakout-VS1063:1X10, symbol SparkFun_MP3_Breakout-VS1063-eagle-import:M10"
- added LED1: Power, SparkFun_MP3_Breakout-VS1063:LED-0603, symbol SparkFun-LED:LED0603
- added Q1: 12.288MHz, SparkFun_MP3_Breakout-VS1063:CRYSTAL-SMD-5X3, symbol SparkFun_MP3_Breakout-VS1063-eagle-import:CRYSTAL5X3
- added U$12: 1.8V, SparkFun_MP3_Breakout-VS1063:SC70, symbol SparkFun_MP3_Breakout-VS1063-eagle-import:V_REG_LDOSMD
- added U$2: 2.8V, SparkFun_MP3_Breakout-VS1063:SC70, symbol SparkFun_MP3_Breakout-VS1063-eagle-import:V_REG_LDOSMD
- added U1: 3.3V, SparkFun_MP3_Breakout-VS1063:SOT23-5, symbol SparkFun_MP3_Breakout-VS1063-eagle-import:V_REG_LDOSMD
- added U2: VS1053, SparkFun_MP3_Breakout-VS1063:LQFP-48, symbol SparkFun_MP3_Breakout-VS1063-eagle-import:VS1033
- C1: renamed from C5; footprint SparkFun-Capacitors:EIA3216 -> SparkFun_MP3_Breakout-VS1063:EIA3216
- C10: renamed from C19; footprint SparkFun-Capacitors:0402-CAP -> SparkFun_MP3_Breakout-VS1063:0402-CAP
- C11: renamed from C20; footprint SparkFun-Capacitors:0402-CAP -> SparkFun_MP3_Breakout-VS1063:0402-CAP
- C12: renamed from C21; footprint SparkFun-Capacitors:0402-CAP -> SparkFun_MP3_Breakout-VS1063:0402-CAP
- C13: renamed from C7; footprint SparkFun-Capacitors:0402-CAP -> SparkFun_MP3_Breakout-VS1063:0402-CAP
- C14: renamed from C11; footprint SparkFun-Capacitors:0402-CAP -> SparkFun_MP3_Breakout-VS1063:0402-CAP
- C15: renamed from C12; footprint SparkFun-Capacitors:0402-CAP -> SparkFun_MP3_Breakout-VS1063:0402-CAP
- C16: renamed from C15; footprint SparkFun-Capacitors:0402-CAP -> SparkFun_MP3_Breakout-VS1063:0402-CAP
- C17: renamed from C1; footprint SparkFun-Capacitors:0402-CAP -> SparkFun_MP3_Breakout-VS1063:0402-CAP
- C18: renamed from C2; footprint SparkFun-Capacitors:0402-CAP -> SparkFun_MP3_Breakout-VS1063:0402-CAP
- C19: renamed from C3; footprint SparkFun-Capacitors:0402-CAP -> SparkFun_MP3_Breakout-VS1063:0402-CAP
- C2: renamed from C9; footprint SparkFun-Capacitors:0402-CAP -> SparkFun_MP3_Breakout-VS1063:0402-CAP
- C20: renamed from C16; footprint SparkFun-Capacitors:0402-CAP -> SparkFun_MP3_Breakout-VS1063:0402-CAP
- C21: renamed from C17; footprint SparkFun-Capacitors:0402-CAP -> SparkFun_MP3_Breakout-VS1063:0402-CAP
- C22: renamed from C18; footprint SparkFun-Capacitors:0402-CAP -> SparkFun_MP3_Breakout-VS1063:0402-CAP
- C23, C24: footprint SparkFun-Capacitors:0402-CAP -> SparkFun_MP3_Breakout-VS1063:0402-CAP
- C3: renamed from C13; footprint SparkFun-Capacitors:0402-CAP -> SparkFun_MP3_Breakout-VS1063:0402-CAP
- C4: renamed from C6; footprint SparkFun-Capacitors:EIA3216 -> SparkFun_MP3_Breakout-VS1063:EIA3216
- C5: renamed from C8; footprint SparkFun-Capacitors:0402-CAP -> SparkFun_MP3_Breakout-VS1063:0402-CAP
- C6: renamed from C4; footprint SparkFun-Capacitors:EIA3216 -> SparkFun_MP3_Breakout-VS1063:EIA3216
- C7: renamed from C10; footprint SparkFun-Capacitors:0402-CAP -> SparkFun_MP3_Breakout-VS1063:0402-CAP
- C8: renamed from C14; footprint SparkFun-Capacitors:0402-CAP -> SparkFun_MP3_Breakout-VS1063:0402-CAP
- C9: renamed from C22; footprint SparkFun-Capacitors:0402-CAP -> SparkFun_MP3_Breakout-VS1063:0402-CAP
- JP2: footprint SparkFun-Connectors:1X10_LOCK -> SparkFun_MP3_Breakout-VS1063:1X10
- JP3: footprint SparkFun-Connectors:1X07 -> SparkFun_MP3_Breakout-VS1063:1X07
- JP4: footprint SparkFun-Capacitors:SJ_2S -> SparkFun_MP3_Breakout-VS1063:SJ_2S
- R1: renamed from R6; footprint SparkFun-Capacitors:0402-RES -> SparkFun_MP3_Breakout-VS1063:0402-RES
- R10: renamed from R3; footprint SparkFun-Resistors:0402-RES -> SparkFun_MP3_Breakout-VS1063:0402-RES
- R11: renamed from R4; footprint SparkFun-Capacitors:0402-RES -> SparkFun_MP3_Breakout-VS1063:0402-RES
- R12: renamed from R14; footprint SparkFun-Capacitors:0402-RES -> SparkFun_MP3_Breakout-VS1063:0402-RES
- R13: renamed from R15; footprint SparkFun-Capacitors:0402-RES -> SparkFun_MP3_Breakout-VS1063:0402-RES
- R14: renamed from R10; footprint SparkFun-Capacitors:0402-RES -> SparkFun_MP3_Breakout-VS1063:0402-RES
- R15: renamed from R9; footprint SparkFun-Capacitors:0402-RES -> SparkFun_MP3_Breakout-VS1063:0402-RES
- R16: renamed from R8; footprint SparkFun-Capacitors:0402-RES -> SparkFun_MP3_Breakout-VS1063:0402-RES
- R17: renamed from R7; footprint SparkFun-Capacitors:0402-RES -> SparkFun_MP3_Breakout-VS1063:0402-RES
- R2: renamed from R5; footprint SparkFun-Capacitors:0402-RES -> SparkFun_MP3_Breakout-VS1063:0402-RES
- R3: renamed from R16; footprint SparkFun-Capacitors:0402-RES -> SparkFun_MP3_Breakout-VS1063:0402-RES
- R4: renamed from R17; footprint SparkFun-Capacitors:0402-RES -> SparkFun_MP3_Breakout-VS1063:0402-RES
- R5: renamed from R2; footprint SparkFun-Capacitors:0402-RES -> SparkFun_MP3_Breakout-VS1063:0402-RES
- R6: renamed from R11; footprint SparkFun-Capacitors:0402-RES -> SparkFun_MP3_Breakout-VS1063:0402-RES
- R7: renamed from R12; footprint SparkFun-Capacitors:0402-RES -> SparkFun_MP3_Breakout-VS1063:0402-RES
- R8: renamed from R1; footprint SparkFun-Capacitors:0402-RES -> SparkFun_MP3_Breakout-VS1063:0402-RES
- R9: renamed from R13; footprint SparkFun-Capacitors:0402-RES -> SparkFun_MP3_Breakout-VS1063:0402-RES
