File: DCI_TP/pcb/DCI_TP.kicad_pcb (KiCad board)
At the start: 2 copper layers, 44 x 38 mm, 52 parts, among them Q1 12.288MHz, U1 3.3V, U2 VS1053

Commit message: Add files via upload
Parts:
- added REF**: OSHW-Logo2_7.3x6mm_SilkScreen, Symbol:OSHW-Logo2_7.3x6mm_SilkScreen, F.Cu at (167.0, 121.0)
